File: pcb/TK44/TK44.kicad_sch (KiCad schematic)
At the start: 108 parts, among them J1 BATT, J2 SWD, J3 USB_C_Receptacle_USB2.0, Q1 AO3407, SW1 MX, SW10 MX, SW11 MX, SW12 MX, SW13 MX, SW14 MX, SW15 MX, SW16 MX, SW17 MX, SW18 MX, SW19 MX, SW2 MX, SW20 MX, SW21 MX, SW22 MX, SW23 MX, SW24 MX, SW25 MX, SW26 MX, SW27 MX, SW28 MX, SW29 MX, SW3 MX, SW30 MX, SW31 MX, SW32 MX, SW33 MX, SW34 MX, SW35 MX, SW36 MX, SW37 MX, SW38 MX, SW39 MX, SW4 MX, SW40 MX, SW41 MX, SW42 MX, SW43 MX, SW44 MX, SW45 SW_DPDT, SW5 MX, SW6 MX, SW7 MX, SW8 MX, SW9 MX, U1 HOLYIOT-18010, U2 MCP73831, U3 XC6220-3.3V

Commit message: 2.0 PCB with battery cutout
Parts:
- added C1 (x2): 10pF, Capacitor_SMD:C_0603_1608Metric_Pad1.08x0.95mm_HandSolder, symbol Device:C_Small
- added C3: 1nF, Capacitor_SMD:C_0603_1608Metric_Pad1.08x0.95mm_HandSolder, symbol Device:C_Small
- added C5 (x2): 4.7uF, Capacitor_SMD:C_0603_1608Metric_Pad1.08x0.95mm_HandSolder, symbol Device:C_Small
- added F1: 500mA, Fuse:Fuse_1206_3216Metric_Pad1.42x1.75mm_HandSolder, symbol Device:Polyfuse_Small
- added J4: BATT_TH, TK44:Battery_Connector_TH, symbol Connector:Conn_01x02_Female
- added R10: 1M, TK44:R_0603, symbol Device:R_Small
- added U4: USBLC6-2SC6, Package_TO_SOT_SMD:SOT-23-6, symbol Power_Protection:USBLC6-2SC6
- J1: footprint TK44:Battery_Connector -> TK44:Battery_Connector_V2
- J2: footprint TK44:Connector_THT_1x4_2.54 -> TK44:Programmer_Conn
- R4: value 810K -> 806K
Connections:
- net DATA+: now also U4.1 (I/O1); no longer J3.A6 (D+), J3.B6 (D+)
- net DATA-: now also U4.3 (I/O2); no longer J3.A7 (D-), J3.B7 (D-)
- net GND: now also J2.2 (Pin_2), C1.1, C1.2, C3.1, C5.2, C5.2, J4.2 (Pin_2), R10.2, U4.2 (GND); no longer J2.1 (Pin_1), R1.2, R2.2
- net VBAT: now also C5.1, J4.1 (Pin_1)
- net VBUS: now also C5.1, F1.2, U4.5 (VBUS); no longer J3.A4 (VBUS), J3.A9 (VBUS), J3.B4 (VBUS), J3.B9 (VBUS)
- net nRF_VDD: now also J2.1 (Pin_1), C1.1; no longer J2.2 (Pin_2)
- net at D46.1 (K), Q1.2 (S), U3.1 (VIN)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: now also C1.2
- net GNDS: now reaches J3.S1 (SHIELD)
- net GNDS: now also R1.2, R2.2, C3.2, R10.1
- new net: F1.1, J3.A4 (VBUS), J3.A9 (VBUS), J3.B4 (VBUS), J3.B9 (VBUS)
- new net USB+: J3.A6 (D+), J3.B6 (D+), U4.6 (I/O1)
- new net USB-: J3.A7 (D-), J3.B7 (D-), U4.4 (I/O2)
- no-connect marks 12 -> 11
Other:
- note added: "ESD protection"
- moved on the sheet: D45, J1, R3

Commit message: Schematic title & attribution
Other:
- company: (none) -> Ladniy & krikun98
- title: (none) -> TK44
Changed lines of the file:
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@@
 (kicad_sch (version 20230121) (generator eeschema)
   (paper "A4")
+  (title_block
+    (title "TK44")
+    (date "2023-03-05")
+    (rev "2.0")
+    (company "Ladniy & krikun98")
+  )
   (junction (at 201.295 38.1) (diameter 0) (color 0 0 0 0)
   )

Commit message: PCBA rework - single-sided PCB
Parts:
- C1, C3, C5: footprint Capacitor_SMD:C_0603_1608Metric_Pad1.08x0.95mm_HandSolder -> Capacitor_SMD:C_0805_2012Metric_Pad1.18x1.45mm_HandSolder
- D45, D47: footprint TK44:LED_0603 -> LED_SMD:LED_0805_2012Metric_Pad1.15x1.40mm_HandSolder
- R1, R10, R2, R3, R4, R5, R6, R7, R8: footprint TK44:R_0603 -> Resistor_SMD:R_0805_2012Metric_Pad1.20x1.40mm_HandSolder
- SWT1: footprint TK44:K2-1187SQ -> Button_Switch_SMD:SW_SPST_EVQP7C
Changed lines of the file:
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@@
       (effects (font (size 1.27 1.27)) (justify left))
     )
-    (property "Footprint" "Capacitor_SMD:C_0603_1608Metric_Pad1.08x0.95mm_HandSolder" (at 80.01 184.785 0)
+    (property "Footprint" "Capacitor_SMD:C_0805_2012Metric_Pad1.18x1.45mm_HandSolder" (at 80.01 184.785 0)
       (effects (font (size 1.27 1.27)) hide)
     )
@@
       (effects (font (size 1.27 1.27)))
     )
-    (property "Footprint" "TK44:R_0603" (at 141.605 184.15 0)
+    (property "Footprint" "Resistor_SMD:R_0805_2012Metric_Pad1.20x1.40mm_HandSolder" (at 141.605 184.15 0)
       (effects (font (size 1.27 1.27)) hide)
     )
@@
       (effects (font (size 1.27 1.27)) (justify left))
     )
-    (property "Footprint" "TK44:R_0603" (at 41.91 140.335 0)
+    (property "Footprint" "Resistor_SMD:R_0805_2012Metric_Pad1.20x1.40mm_HandSolder" (at 41.91 140.335 0)
       (effects (font (size 1.27 1.27)) hide)
     )
@@
       (effects (font (size 1.27 1.27)))
     )
-    (property "Footprint" "TK44:LED_0603" (at 135.255 158.115 90)
+    (property "Footprint" "LED_SMD:LED_0805_2012Metric_Pad1.15x1.40mm_HandSolder" (at 135.255 158.115 90)
       (effects (font (size 1.27 1.27)) hide)
     )
@@
       (effects (font (size 1.27 1.27)))
     )
-    (property "Footprint" "TK44:R_0603" (at 22.86 139.7 0)
+    (property "Footprint" "Resistor_SMD:R_0805_2012Metric_Pad1.20x1.40mm_HandSolder" (at 22.86 139.7 0)
       (effects (font (size 1.27 1.27)) hide)
     )
@@
       (effects (font (size 1.27 1.27)))
     )
-    (property "Footprint" "TK44:R_0603" (at 142.875 158.115 0)
+    (property "Footprint" "Resistor_SMD:R_0805_2012Metric_Pad1.20x1.40mm_HandSolder" (at 142.875 158.115 0)
       (effects (font (size 1.27 1.27)) hide)
     )
@@
       (effects (font (size 1.27 1.27)) (justify left))
     )
-    (property "Footprint" "TK44:R_0603" (at 49.53 140.335 0)
+    (property "Footprint" "Resistor_SMD:R_0805_2012Metric_Pad1.20x1.40mm_HandSolder" (at 49.53 140.335 0)
       (effects (font (size 1.27 1.27)) hide)
     )
@@
       (effects (font (size 1.27 1.27)))
     )
-    (property "Footprint" "TK44:K2-1187SQ" (at 156.845 97.155 0)
+    (property "Footprint" "Button_Switch_SMD:SW_SPST_EVQP7C" (at 156.845 97.155 0)
       (effects (font (size 1.27 1.27)) hide)
     )
@@
       (effects (font (size 1.27 1.27)) (justify right))
     )
-    (property "Footprint" "Capacitor_SMD:C_0603_1608Metric_Pad1.08x0.95mm_HandSolder" (at 113.665 165.735 0)
+    (property "Footprint" "Capacitor_SMD:C_0805_2012Metric_Pad1.18x1.45mm_HandSolder" (at 113.665 165.735 0)
       (effects (font (size 1.27 1.27)) hide)
     )
@@
       (effects (font (size 1.27 1.27)) (justify left))
     )
-    (property "Footprint" "TK44:R_0603" (at 30.48 184.785 0)
+    (property "Footprint" "Resistor_SMD:R_0805_2012Metric_Pad1.20x1.40mm_HandSolder" (at 30.48 184.785 0)
       (effects (font (size 1.27 1.27)) hide)
     )
@@
       (effects (font (size 1.27 1.27)) (justify left))
     )
-    (property "Footprint" "TK44:R_0603" (at 30.48 174.625 0)
+    (property "Footprint" "Resistor_SMD:R_0805_2012Metric_Pad1.20x1.40mm_HandSolder" (at 30.48 174.625 0)
       (effects (font (size 1.27 1.27)) hide)
     )
@@
       (effects (font (size 1.27 1.27)) (justify right))
     )
-    (property "Footprint" "Capacitor_SMD:C_0603_1608Metric_Pad1.08x0.95mm_HandSolder" (at 98.425 165.735 0)
+    (property "Footprint" "Capacitor_SMD:C_0805_2012Metric_Pad1.18x1.45mm_HandSolder" (at 98.425 165.735 0)
       (effects (font (size 1.27 1.27)) hide)
     )
@@
       (effects (font (size 1.27 1.27)))
     )
-    (property "Footprint" "TK44:R_0603" (at 111.125 184.15 0)
+    (property "Footprint" "Resistor_SMD:R_0805_2012Metric_Pad1.20x1.40mm_HandSolder" (at 111.125 184.15 0)
       (effects (font (size 1.27 1.27)) hide)
     )
@@
       (effects (font (size 1.27 1.27)) (justify left))
     )
-    (property "Footprint" "TK44:R_0603" (at 45.72 184.785 0)
+    (property "Footprint" "Resistor_SMD:R_0805_2012Metric_Pad1.20x1.40mm_HandSolder" (at 45.72 184.785 0)
       (effects (font (size 1.27 1.27)) hide)
     )
@@
       (effects (font (size 1.27 1.27)))
     )
-    (property "Footprint" "TK44:LED_0603" (at 103.505 184.15 90)
+    (property "Footprint" "LED_SMD:LED_0805_2012Metric_Pad1.15x1.40mm_HandSolder" (at 103.505 184.15 90)
       (effects (font (size 1.27 1.27)) hide)
     )
@@
       (effects (font (size 1.27 1.27)))
     )
-    (property "Footprint" "Capacitor_SMD:C_0603_1608Metric_Pad1.08x0.95mm_HandSolder" (at 22.86 142.875 0)
+    (property "Footprint" "Capacitor_SMD:C_0805_2012Metric_Pad1.18x1.45mm_HandSolder" (at 22.86 142.875 0)
       (effects (font (size 1.27 1.27)) hide)
     )
@@
       (effects (font (size 1.27 1.27)) (justify left))
     )
-    (property "Footprint" "Capacitor_SMD:C_0603_1608Metric_Pad1.08x0.95mm_HandSolder" (at 58.42 184.785 0)
+    (property "Footprint" "Capacitor_SMD:C_0805_2012Metric_Pad1.18x1.45mm_HandSolder" (at 58.42 184.785 0)
       (effects (font (size 1.27 1.27)) hide)
     )

Commit message: Move reset/LEDs, round pads
Parts:
- SWT1: footprint Button_Switch_SMD:SW_SPST_EVQP7C -> TK44:SW_SPST_EVQP7C
Changed lines of the file:
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@@
       (effects (font (size 1.27 1.27)))
     )
-    (property "Footprint" "Button_Switch_SMD:SW_SPST_EVQP7C" (at 156.845 97.155 0)
+    (property "Footprint" "TK44:SW_SPST_EVQP7C" (at 156.845 97.155 0)
       (effects (font (size 1.27 1.27)) hide)
     )
